File: BooskieBadge.kicad_sch (KiCad schematic)
At the start: 32 parts, among them J1 TC2030, U1 nRF52840, Y1 32MHz

Commit message: pcb first pass
Parts:
- AE1: footprint (none) -> BooskieBadge:2.4GHz-meander-antenna-v2
- AE2: footprint (none) -> BooskieBadge:NFC_ANTENNA
- C1, C10, C11, C12, C14, C17, C18, C19, C2, C29, C3, C33, C34, C35, C6, C7, C8, C9: footprint (none) -> Capacitor_SMD:C_0402_1005Metric
- C13, C15, C16, C4, C5: footprint (none) -> Capacitor_SMD:C_0603_1608Metric
- L1, L2: footprint (none) -> Inductor_SMD:L_0402_1005Metric
- L3, L5: footprint (none) -> Inductor_SMD:L_0603_1608Metric
- Y1: footprint (none) -> Crystal:Crystal_SMD_2016-4Pin_2.0x1.6mm
Changed lines of the file:
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@@
 			)
 		)
-		(property "Footprint" ""
+		(property "Footprint" "Capacitor_SMD:C_0402_1005Metric"
 			(at 63.5 29.21 0)
 			(effects
@@
 			)
 		)
-		(property "Footprint" ""
+		(property "Footprint" "Capacitor_SMD:C_0402_1005Metric"
 			(at 177.8 31.75 0)
 			(effects
@@
 			)
 		)
-		(property "Footprint" ""
+		(property "Footprint" "Inductor_SMD:L_0402_1005Metric"
 			(at 46.99 71.12 0)
 			(effects
@@
 			)
 		)
-		(property "Footprint" ""
+		(property "Footprint" "Capacitor_SMD:C_0603_1608Metric"
 			(at 106.68 31.75 0)
 			(effects
@@
 			)
 		)
-		(property "Footprint" ""
+		(property "Footprint" "Capacitor_SMD:C_0402_1005Metric"
 			(at 154.94 31.75 0)
 			(effects
@@
 			)
 		)
-		(property "Footprint" ""
+		(property "Footprint" "Crystal:Crystal_SMD_2016-4Pin_2.0x1.6mm"
 			(at 40.64 116.84 0)
 			(effects
@@
 			)
 		)
-		(property "Footprint" ""
+		(property "Footprint" "Capacitor_SMD:C_0603_1608Metric"
 			(at 33.02 46.99 0)
 			(effects
@@
 			)
 		)
-		(property "Footprint" ""
+		(property "Footprint" "Capacitor_SMD:C_0402_1005Metric"
 			(at 82.55 17.78 0)
 			(effects
@@
 			)
 		)
-		(property "Footprint" ""
+		(property "Footprint" "Capacitor_SMD:C_0402_1005Metric"
 			(at 154.94 72.39 0)
 			(effects
@@
 			)
 		)
-		(property "Footprint" ""
+		(property "Footprint" "Capacitor_SMD:C_0402_1005Metric"
 			(at 166.37 31.75 0)
 			(effects
@@
 			)
 		)
-		(property "Footprint" ""
+		(property "Footprint" "Capacitor_SMD:C_0402_1005Metric"
 			(at 41.91 46.99 0)
 			(effects
@@
 			)
 		)
-		(property "Footprint" ""
+		(property "Footprint" "Capacitor_SMD:C_0402_1005Metric"
 			(at 38.1 76.2 0)
 			(effects
@@
 			)
 		)
-		(property "Footprint" ""
+		(property "Footprint" "Inductor_SMD:L_0402_1005Metric"
 			(at 96.52 34.29 0)
 			(effects
@@
 			)
 		)
-		(property "Footprint" ""
+		(property "Footprint" "Capacitor_SMD:C_0402_1005Metric"
 			(at 31.75 111.76 0)
 			(effects
@@
 			)
 		)
-		(property "Footprint" ""
+		(property "Footprint" "BooskieBadge:NFC_ANTENNA"
 			(at 167.64 76.2 0)
 			(effects
@@
 			)
 		)
-		(property "Footprint" ""
+		(property "Footprint" "Capacitor_SMD:C_0603_1608Metric"
 			(at 21.59 46.99 0)
 			(effects
@@
 			)
 		)
-		(property "Footprint" ""
+		(property "Footprint" "Capacitor_SMD:C_0402_1005Metric"
 			(at 52.07 76.2 0)
 			(effects
@@
 			)
 		)
-		(property "Footprint" ""
+		(property "Footprint" "Inductor_SMD:L_0603_1608Metric"
 			(at 96.52 40.64 0)
 			(effects
@@
 			)
 		)
-		(property "Footprint" ""
+		(property "Footprint" "Capacitor_SMD:C_0402_1005Metric"
 			(at 53.34 46.99 0)
 			(effects
@@
 			)
 		)
-		(property "Footprint" ""
+		(property "Footprint" "Capacitor_SMD:C_0603_1608Metric"
 			(at 132.08 31.75 0)
 			(effects
@@
 			)
 		)
-		(property "Footprint" ""
+		(property "Footprint" "Capacitor_SMD:C_0402_1005Metric"
 			(at 31.75 121.92 0)
 			(effects
@@
 			)
 		)
-		(property "Footprint" ""
+		(property "Footprint" "BooskieBadge:2.4GHz-meander-antenna-v2"
 			(at 24.13 64.77 0)
 			(effects
@@
 			)
 		)
-		(property "Footprint" ""
+		(property "Footprint" "Capacitor_SMD:C_0402_1005Metric"
 			(at 119.38 31.75 0)
 			(effects
@@
 			)
 		)
-		(property "Footprint" ""
+		(property "Footprint" "Inductor_SMD:L_0603_1608Metric"
 			(at 38.1 30.48 0)
 			(effects
@@
 			)
 		)
-		(property "Footprint" ""
+		(property "Footprint" "Capacitor_SMD:C_0402_1005Metric"
 			(at 143.51 82.55 0)
 			(effects
@@
 			)
 		)
-		(property "Footprint" ""
+		(property "Footprint" "Capacitor_SMD:C_0402_1005Metric"
 			(at 154.94 82.55 0)
 			(effects
@@
 			)
 		)
-		(property "Footprint" ""
+		(property "Footprint" "Capacitor_SMD:C_0402_1005Metric"
 			(at 143.51 72.39 0)
 			(effects
@@
 			)
 		)
-		(property "Footprint" ""
+		(property "Footprint" "Capacitor_SMD:C_0603_1608Metric"
 			(at 143.51 31.75 0)
 			(effects
@@
 			)
 		)
-		(property "Footprint" ""
+		(property "Footprint" "Capacitor_SMD:C_0402_1005Metric"
 			(at 24.13 76.2 0)
 			(effects
@@
 			)
 		)
-		(property "Footprint" ""
+		(property "Footprint" "Capacitor_SMD:C_0402_1005Metric"
 			(at 63.5 24.13 0)
 			(effects
@@
 	)
 	(sheet
-		(at 227.33 124.46)
+		(at 142.24 158.75)
 		(size 26.67 16.51)
 		(exclude_from_sim no)
@@
 		)
 		(property "Sheetname" "Display"
-			(at 227.33 123.7484 0)
+			(at 142.24 158.0384 0)
 			(effects
 				(font
@@
 		)
 		(property "Sheetfile" "Display.kicad_sch"
-			(at 227.33 141.5546 0)
+			(at 142.24 175.8446 0)
 			(effects
 				(font

Commit message: screwing around with ports and stuff
Parts:
- added BT1: Battery_Cell, BooskieBadge:BAT_HOLDER_2032SMD, symbol Device:Battery_Cell
- added J3: USB_C_Receptacle_PCB_Edge, BooskieBadge:USB_C_PCB_receptacle_24pin_1mm-cutout, symbol BooskieBadge:USB_C_Receptacle_PCB_Edge
- added J4: USB_A_PCB_Edge_receptacle, BooskieBadge:USB_A_PCB_Edge_receptacle, symbol BooskieBadge:USB_A_PCB_Edge_receptacle
- added R1, R4: 5.1k, Resistor_SMD:R_0402_1005Metric, symbol Device:R_Small
- added U2: USBLC6-2P6, Package_TO_SOT_SMD:SOT-666, symbol Power_Protection:USBLC6-2P6
- added U3: SAOV1.69BIS, BooskieBadge:Simple_Addon_v2-BADGE-2x3, symbol BooskieBadge:SAOV1.69BIS
Connections:
- net +BATT: now also BT1.1 (+)
- net GND: now also BT1.2 (-), J3.A1 (GND), J3.A12 (GND), J3.B1 (GND), J3.B12 (GND), J4.4 (GND), R1.1, R4.1, U2.2 (GND), U3.2 (GND)
- net VBUS: now also J3.A4 (VBUS), J3.A9 (VBUS), J3.B4 (VBUS), J3.B9 (VBUS), J4.1 (VBUS), U2.5 (VBUS)
- net VDD: now also U3.1 (VCC)
- net at U1.A10 (AIN5/P0.29): now also U3.6 (GPIO2)
- net D-: now reaches U1.AD4 (D-)
- net D-: now also U2.3 (I/O2)
- net D+: now reaches U1.AD6 (D+)
- net D+: now also U2.1 (I/O1)
- net at U1.B11 (AIN4/P0.28): now also U3.5 (GPIO1)
- net SDA: now reaches U1.G1 (P0.26)
- net SDA: now also U3.3 (SDA)
- net SCL: now reaches U1.H2 (P0.27)
- net SCL: now also U3.4 (SCL)
- new net: J3.B5 (CC2), R4.2
- new net: J3.A5 (CC1), R1.2
- new net D_N: J3.A7 (D-), J3.B7 (D-), J4.2 (D-), U2.4 (I/O2)
- new net D_P: J3.A6 (D+), J3.B6 (D+), J4.3 (D+), U2.6 (I/O1)

Commit message: rtc crystal
Parts:
- added C36, C37: 12pF, Capacitor_SMD:C_0402_1005Metric, symbol Device:C_Small
- added Y2: 32.768 kHz, Crystal:Crystal_SMD_3215-2Pin_3.2x1.5mm, symbol Device:Crystal_Small
- Y1: symbol Device:Crystal_Small -> Device:Crystal_GND24_Small
Connections:
- net GND: now also C36.2, C37.2
- net at C2.2, U1.B24 (XC1): now also Y1.3; no longer Y1.2
- net at U1.D2 (XL1/P0.00): now also C36.1, Y2.2
- net at U1.F2 (XL2/P0.01): now also C37.1, Y2.1
- new net: Y1.2 (G), Y1.4 (G)
- no-connect marks 1 -> 2
Other:
- moved on the sheet: AE2, C29, C33, C34, C35

Commit message: time-of-flight, plus usb, plus li-ion option
Parts:
- removed J3: USB_C_Receptacle_PCB_Edge, BooskieBadge:USB_C_PCB_receptacle_24pin_1mm-cutout, symbol BooskieBadge:USB_C_Receptacle_PCB_Edge
- removed J4: USB_A_PCB_Edge_receptacle, BooskieBadge:USB_A_PCB_Edge_receptacle, symbol BooskieBadge:USB_A_PCB_Edge_receptacle
- added D4: LED, BooskieBadge:LED_LB Q39G-L2OO-35-1_OSR, symbol Device:LED
- added J3: USB_C_Receptacle_USB2.0_16P, Connector_USB:USB_C_Receptacle_JAE_DX07S016JA1R1500, symbol Connector:USB_C_Receptacle_USB2.0_16P
- added J4: JST_PH, Connector_JST:JST_PH_S2B-PH-K_1x02_P2.00mm_Horizontal, symbol Connector:Conn_01x02_Socket
- added J5: Conn_01x04, Connector_JST:JST_SH_SM04B-SRSS-TB_1x04-1MP_P1.00mm_Horizontal, symbol Connector_Generic:Conn_01x04
- added R10, R5, R6, R7, R8, R9: 10k, Resistor_SMD:R_0402_1005Metric, symbol Device:R_Small
- added R11, R12: 5.1k, Resistor_SMD:R_0402_1005Metric, symbol Device:R_Small
- added SW1: RST, Button_Switch_SMD:SW_Push_1P1T_NO_CK_KMR2, symbol Switch:SW_Push
- added SW2: USR, Button_Switch_SMD:SW_Push_1P1T_NO_CK_KMR2, symbol Switch:SW_Push
- added U4: MCP73831T-2ACI/OT, BooskieBadge:SOT-23-5_MC_MCH, symbol BooskieBadge:MCP73831T-2ACI_OT
- added U5: VL53L1CXV0FY1, Sensor_Distance:ST_VL53L1x, symbol Sensor_Distance:VL53L1CXV0FY1
Connections:
- net +BATT: now also J4.1 (Pin_1), U4.3 (VBAT); no longer L5.2
- net D_N: now also J3.A7 (D-), J3.B7 (D-)
- net D_P: now also J3.A6 (D+), J3.B6 (D+)
- net GND: now also J3.A1 (GND), J3.A12 (GND), J3.B1 (GND), J3.B12 (GND), J3.S1 (SHIELD), J4.2 (Pin_2), J5.4 (Pin_4), R10.1, R11.2, R9.1, U4.2 (VSS), U5.12 (GND), U5.2 (AVSSVCSEL), U5.3 (GND), U5.4 (GND), U5.6 (GND)
- net SCL: now also J5.1 (Pin_1), R5.1, U5.10 (SCL)
- net SDA: now also J5.2 (Pin_2), R6.1, U5.9 (SDA)
- net VBUS: now also J3.A4 (VBUS), J3.A9 (VBUS), J3.B4 (VBUS), J3.B9 (VBUS), R12.2, U4.4 (VDD)
- net VDD: now also J5.3 (Pin_3), R5.2, R6.2, R7.2, R8.2, U5.1 (AVDDVCSEL), U5.11 (AVDD)
- net ~{RST}: now also SW1.1
- net at U1.A10 (AIN5/P0.29): no longer U3.6 (GPIO2)
- net SAO_GP2: now reaches U1.A12 (AIN0/P0.02)
- net SAO_GP2: now also U3.6 (GPIO2)
- net at U1.AB2 (DCCH): now also L5.2
- net at U1.B11 (AIN4/P0.28): no longer U3.5 (GPIO1)
- net SAO_GP1: now reaches U1.J1 (AIN2/P0.04)
- net SAO_GP1: now also U3.5 (GPIO1)
- net TOF_SHDN: now reaches U1.L1 (P0.06)
- net TOF_SHDN: now also R7.1, U5.5 (XSHUT)
- net TOF_GP1: now reaches U1.N1 (P0.08)
- net TOF_GP1: now also R8.1, U5.7 (GPIO1)
- net at U1.U1 (TRACEDATA1/P0.12): now also SW2.1
- net at R4.2: now also J3.B5 (CC2)
- net at R1.2: now also J3.A5 (CC1)
- new net: R10.2, SW2.2
- new net: D4.2 (A), R12.1
- new net: D4.1 (K), U4.1 (STAT)
- new net: R11.1, U4.5 (PROG)
- new net: R9.2, SW1.2
- no-connect marks 2 -> 1
Other:
- moved on the sheet: AE2, BT1, C29, C33, C34, C35, C36, C37, L5, R1, R4, U2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
