File: BooskieBadge.kicad_pcb (KiCad board)
At the start: 4 copper layers, 79 x 44.2 mm, 77 parts, among them J1 TC2030, J2 SFV24R-2STE1HLF, J3 USB_C_Receptacle_USB2.0_16P, J4 JST_PH, J5 Conn_01x04, Q1 Si1308EDL, SW1 RST, SW2 USR, U1 nRF52840, U2 USBLC6-2P6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

Commit message: board edges
Other:
- board size 79 x 44.2 mm -> 88.3 x 44.6 mm
Changed lines of the file:
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@@
 		(tags "USB C Type-C Receptacle SMD USB 2.0")
 		(property "Reference" "J3"
-			(at 0 5 0)
+			(at -6.537653 -1.062347 180)
 			(layer "B.SilkS")
 			(effects
@@
 	)
 	(gr_rect
+		(start 65 101.5)
+		(end 144 138.2)
+		(stroke
+			(width 0.3)
+			(type default)
+		)
+		(fill no)
+		(layer "B.SilkS")
+	)
+	(gr_rect
 		(start 67.637653 101.362347)
 		(end 146.637653 138.062347)
@@
 	)
 	(gr_line
-		(start 113.137653 138.112347)
-		(end 101.137653 138.112347)
+		(start 112.887653 138.5)
+		(end 100.5 138.5)
 		(stroke
 			(width 0.05)
@@
 	)
 	(gr_line
-		(start 67.637653 138.112347)
-		(end 67.637653 100.612347)
+		(start 148.819312 110.790698)
+		(end 148.819312 128.709302)
+		(stroke
+			(width 0.05)
+			(type default)
+		)
+		(layer "Edge.Cuts")
+	)
+	(gr_line
+		(start 62.27297 136.5)
+		(end 62.27297 100.612347)
 		(stroke
 			(width 0.05)
@@
 	)
 	(gr_arc
-		(start 67.637653 100.612347)
-		(mid 69.614682 95.839376)
-		(end 74.387653 93.862347)
+		(start 62.27297 100.612347)
+		(mid 64.25 95.839379)
+		(end 69.02297 93.862347)
 		(stroke
 			(width 0.05)
@@
 	)
 	(gr_line
-		(start 109.137653 96.862347)
-		(end 115.137653 96.862347)
+		(start 108.75 96.862347)
+		(end 114.75 96.862347)
 		(stroke
 			(width 0.05)
@@
 	)
 	(gr_line
-		(start 146.637653 94.612347)
-		(end 146.637653 138.112347)
+		(start 150.569312 95.862347)
+		(end 150.569312 106.709302)
 		(stroke
 			(width 0.05)
@@
 	)
 	(gr_line
-		(start 101.137653 138.112347)
-		(end 67.637653 138.112347)
+		(start 100.5 138.5)
+		(end 63.77297 138.5)
 		(stroke
 			(width 0.05)
@@
 	)
 	(gr_line
-		(start 74.410624 93.862347)
+		(start 69.02297 93.862347)
 		(end 107.137653 93.862347)
 		(stroke
@@
 	)
 	(gr_line
-		(start 146.637653 138.112347)
-		(end 113.137653 138.112347)
+		(start 148.569312 138.5)
+		(end 112.887653 138.5)
 		(stroke
 			(width 0.05)
@@
 	)
 	(gr_line
-		(start 115.137653 100.362347)
-		(end 99.137653 100.362347)
+		(start 114.75 100.362347)
+		(end 98.75 100.362347)
+		(stroke
+			(width 0.05)
+			(type default)
+		)
+		(layer "Edge.Cuts")
+	)
+	(gr_line
+		(start 150.569312 132.790698)
+		(end 150.569312 136.5)
 		(stroke
 			(width 0.05)
@@
 	)
 	(gr_arc
-		(start 105.137653 96.862347)
-		(mid 107.137653 94.862347)
-		(end 109.137653 96.862347)
+		(start 150.569312 106.709302)
+		(mid 150.5 107.231262)
+		(end 150.29687 107.717044)
 		(stroke
 			(width 0.05)
@@
 	)
 	(gr_arc
-		(start 99.137653 100.362347)
-		(mid 97.387653 98.612347)
-		(end 99.137653 96.862347)
+		(start 104.75 96.862347)
+		(mid 106.75 94.862347)
+		(end 108.75 96.862347)
 		(stroke
 			(width 0.05)
@@
 	)
 	(gr_arc
-		(start 115.137653 96.862347)
-		(mid 116.887653 98.612347)
-		(end 115.137653 100.362347)
+		(start 149.091754 129.717044)
+		(mid 148.888623 129.231262)
+		(end 148.819312 128.709302)
+		(stroke
+			(width 0.05)
+			(type default)
+		)
+		(layer "Edge.Cuts")
+	)
+	(gr_arc
+		(start 150.29687 131.782956)
+		(mid 150.500001 132.268738)
+		(end 150.569312 132.790698)
+		(stroke
+			(width 0.05)
+			(type default)
+		)
+		(layer "Edge.Cuts")
+	)
+	(gr_arc
+		(start 64.27297 138.5)
+		(mid 62.858757 137.914213)
+		(end 62.27297 136.5)
+		(stroke
+			(width 0.05)
+			(type default)
+		)
+		(layer "Edge.Cuts")
+	)
+	(gr_line
+		(start 149.091754 129.717044)
+		(end 150.29687 131.782956)
+		(stroke
+			(width 0.05)
+			(type default)
+		)
+		(layer "Edge.Cuts")
+	)
+	(gr_arc
+		(start 98.75 100.362347)
+		(mid 97 98.612347)
+		(end 98.75 96.862347)
+		(stroke
+			(width 0.05)
+			(type default)
+		)
+		(layer "Edge.Cuts")
+	)
+	(gr_line
+		(start 149.091754 109.782956)
+		(end 150.29687 107.717044)
+		(stroke
+			(width 0.05)
+			(type default)
+		)
+		(layer "Edge.Cuts")
+	)
+	(gr_arc
+		(start 150.569312 136.5)
+		(mid 149.983509 137.914183)
+		(end 148.569312 138.5)
+		(stroke
+			(width 0.05)
+			(type default)
+		)
+		(layer "Edge.Cuts")
+	)
+	(gr_arc
+		(start 148.569312 93.862347)
+		(mid 149.983509 94.448136)
+		(end 150.569312 95.862347)
+		(stroke
+			(width 0.05)
+			(type default)
+		)
+		(layer "Edge.Cuts")
+	)
+	(gr_arc
+		(start 148.819312 110.790698)
+		(mid 148.888624 110.268738)
+		(end 149.091754 109.782956)
+		(stroke
+			(width 0.05)
+			(type default)
+		)
+		(layer "Edge.Cuts")
+	)
+	(gr_arc
+		(start 114.75 96.862347)
+		(mid 116.5 98.61235)
+		(end 114.75 100.362347)
 		(stroke
 			(width 0.05)
@@
 	(gr_line
 		(start 107.137653 93.862347)
-		(end 145.887653 93.862347)
+		(end 148.569312 93.862347)
 		(stroke
 			(width 0.05)
@@
 	)
 	(gr_line
-		(start 99.137653 96.862347)
-		(end 105.137653 96.862347)
-		(stroke
-			(width 0.05)
-			(type default)
-		)
-		(layer "Edge.Cuts")
-	)
-	(gr_arc
-		(start 145.887653 93.862347)
-		(mid 146.417983 94.082017)
-		(end 146.637653 94.612347)
+		(start 98.75 96.862347)
+		(end 104.75 96.862347)
 		(stroke
 			(width 0.05)
@@
 	)
 	(segment
-		(start 94.387653 136.848267)
-		(end 95.658933 136.848267)
-		(width 0.2)
-		(layer "F.Cu")
-		(net 3)
-	)
-	(segment
 		(start 96.892653 130.382347)
 		(end 111.762653 130.382347)
@@
 	)
 	(segment
-		(start 95.637653 136.848267)
-		(end 95.651733 136.848267)
+		(start 95.651733 136.848267)
+		(end 96.137653 136.362347)
 		(width 0.2)
 		(layer "F.Cu")
@@
 	)
 	(segment
-		(start 95.651733 136.848267)
-		(end 96.137653 136.362347)
-		(width 0.2)
-		(layer "F.Cu")
-		(net 3)
-	)
-	(segment
 		(start 117.117653 130.382347)
 		(end 111.762653 130.382347)
@@
 		(start 118.937653 128.562347)
 		(end 117.117653 130.382347)
+		(width 0.2)
+		(layer "F.Cu")
+		(net 3)
+	)
+	(segment
+		(start 94.387653 136.848267)
+		(end 95.651733 136.848267)
 		(width 0.2)
 		(layer "F.Cu")
@@
 	)
 	(via
-		(at 127.387653 135.862347)
+		(at 127.387653 136.25)
 		(size 0.4)
 		(drill 0.3)
